Commit message: field world and one wheel

File: src/simulation/models/common/ground_plane.xacro (robot description, xacro)
@@ -18,7 +18,8 @@
         </geometry>
         <material>
-            <ambient>0.8 0.8 0.8 1</ambient>
-            <diffuse>0.8 0.8 0.8 1</diffuse>
-            <specular>0.8 0.8 0.8 1</specular>
+            <script>
+                <uri>file://media/materials/scripts/gazebo.material</uri>
+                <name>Gazebo/Grey</name>
+            </script>
         </material>
         </visual>

File: src/simulation/models/rover/rover.xacro (robot description, xacro)
@@ -2,10 +2,11 @@
 <xacro:macro name="rover">
 <xacro:include filename="$(env MODELS_DIR)/common/utils.xacro" />
-<xacro:include filename="$(env MODELS_DIR)/rover/sslidar.xacro" />
+<xacro:include filename="sslidar.xacro" />
+<xacro:include filename="wheel.xacro" />
 <xacro:property name="robot_side_len" value="0.2" />
 <xacro:property name="robot_mass" value="2" />
 <link name="base">
     <visual name="base_visual">
-        <origin  xyz="0 0 ${-robot_side_len/2}" rpy="${pi / 2} 0 ${pi / 2}"/>
+        <origin  xyz="0 0 0" rpy="0 0 0"/>
         <geometry>
             <box size="${robot_side_len} ${robot_side_len} ${robot_side_len}" />
@@ -29,5 +30,5 @@
     <visual name="base_visual">
         <geometry>
-            <sphere radius="0.08"/>
+            <sphere radius="${robot_side_len / 2 + 0.025}"/>
             <material name="red">
                 <color rgba="1.0 0 0 1.0"/>
@@ -40,4 +41,5 @@
     <child link="base_weight"/>
 </joint>
+<xacro:wheel index="0" xyz="1 0 0" axis="0 1 0"/>
 <!-- CAMERA BLOCK-->
 <link name="camera"></link>
@@ -78,4 +80,12 @@
   </plugin>
 </gazebo>
+<gazebo>
+    <plugin
+        filename="gz-sim-joint-state-publisher-system"
+        name="gz::sim::systems::JointStatePublisher">
+        <topic>joint_states</topic> <!--from <ros><remapping> -->
+        <joint_name>wheel_0_joint</joint_name>
+  </plugin>
+</gazebo>
 </xacro:macro>
 </include>

File: src/simulation/models/worlds/field/field.sdf.xacro (robot description, xacro)
@@ -1,8 +1,21 @@
 <?xml version="1.0" ?>
 <sdf xmlns:xacro="http://www.ros.org/wiki/xacro" version="1.10">
-<world name="plane_world">
+<world name="field_world">
 <xacro:include filename="$(env MODELS_DIR)/common/plugins.xacro" />
 <xacro:include filename="$(env MODELS_DIR)/common/simple_light.xacro" />
-<xacro:include filename="$(env MODELS_DIR)/common/ground_plane.xacro" />
+<include>
+    <uri>file:/$(env MODELS_DIR)/objects/field</uri>
+    <pose>0 0 0 ${-pi/2} 0 0</pose>
+</include>
+<include>
+    <name>pole_1</name>
+    <uri>file:/$(env MODELS_DIR)/objects/marker</uri>
+    <pose>1 0 0 0 0 0</pose>
+</include>
+<include>
+    <name>pole_2</name>
+    <uri>file:/$(env MODELS_DIR)/objects/marker</uri>
+    <pose>0 1 0 0 0 0</pose>
+</include>
 <model name='rover'>
     <include>
