Commit message: working gz system

File: src/simulation/models/common/utils.xacro (robot description, xacro)
@@ -1,3 +1,7 @@
 <include xmlns:xacro="http://www.ros.org/wiki/xacro">
+<xacro:property
+  name="gazebo_systems_lib_dir"
+  value="$(env PROJECT_ROOT)/install/gazebo_systems/lib/gazebo_systems"
+/>
 <xacro:macro name="primitive" params="name *origin *geometry">
   <visual name="${name}">

File: src/simulation/models/worlds/plane.sdf.xacro (robot description, xacro)
@@ -5,4 +5,5 @@
 <xacro:include filename="$(env MODELS_DIR)/common/simple_light.xacro" />
 <xacro:include filename="$(env MODELS_DIR)/common/ground_plane.xacro" />
+<xacro:include filename="$(env MODELS_DIR)/common/utils.xacro" />
 <model name='rover'>
     <include>
@@ -11,4 +12,14 @@
     </include>
 </model>
+<plugin
+    filename="${gazebo_systems_lib_dir}/libDoorButtonSystem.so"
+    name="gz::sim::v8::systems::DoorButtonSystem">
+</plugin>
+<!--
+<plugin filename="gz-sim-python-system-loader-system" name="gz::sim::systems::PythonSystemLoader">
+    <module_name>systems/door.py</module_name>
+    <force>100</force>
+</plugin>
+-->
 </world>
 </sdf>

Commit message: add door and switch

File: src/simulation/models/common/utils.xacro (robot description, xacro)
@@ -4,13 +4,35 @@
   value="$(env PROJECT_ROOT)/install/gazebo_systems/lib/gazebo_systems"
 />
-<xacro:macro name="primitive" params="name *origin *geometry">
-  <visual name="${name}">
-    <xacro:insert_block name="origin"/>
-    <xacro:insert_block name="geometry"/>
+<xacro:macro name="cuboid_form" params="a b c">
+    <geometry>
+      <box><size>${a} ${b} ${c}</size></box>
+    </geometry>
+</xacro:macro>
+<xacro:macro name="cuboid" params="name a b c weight pose:='0 0 0 0 0 0' color:=Yellow is_kinematic:=false self_collide:=false">
+<link name="${name}">
+  <self_collide>${self_collide}</self_collide>
+  <kinematic>${is_kinematic}</kinematic>
+  <pose>${pose}</pose>
+  <collision name="${name}_collision">
+    <xacro:cuboid_form a="${a}" b="${b}" c="${c}"/>
+  </collision>
+  <visual name="${name}_visual">
+    <xacro:cuboid_form a="${a}" b="${b}" c="${c}"/>
+    <material>
+      <script>
+          <uri>file://media/materials/scripts/gazebo.material</uri>
+          <name>Gazebo/${color}</name>
+      </script>
+    </material>
   </visual>
-  <collision name="${name}">
-    <xacro:insert_block name="origin"/>
-    <xacro:insert_block name="geometry"/>
-  </collision>
+  <inertial>
+    <mass>${weight}</mass>
+    <inertia>
+      <ixx>${weight * (a**2 + c**2) / 12}</ixx>
+      <iyy>${weight * (b**2 + c**2) / 12}</iyy>
+      <izz>${weight * (b**2 + a**2) / 12}</izz>
+    </inertia>
+  </inertial>
+</link>
 </xacro:macro>
 </include>

File: src/simulation/models/objects/test/simple_door/model.sdf.xacro (robot description, xacro)
@@ -4,51 +4,8 @@
 <pose>0 0 0 0 0 0</pose>
 <static>false</static>
+<xacro:include filename="$(env MODELS_DIR)/common/utils.xacro" />
 <xacro:property name="base_width" value="1" />
-<link name="door_base">
-  <self_collide>false</self_collide>
-  <kinematic>true</kinematic>
-  <pose>0 0 0 0 0 0</pose>
-  <xacro:macro name="door_base_form">
-    <geometry>
-      <box><size>4 ${base_width} 2</size></box>
-    </geometry>
-  </xacro:macro>
-  <collision name="door_base_collision">
-    <xacro:door_base_form/>
-  </collision>
-  <visual name="door_base_visual">
-    <xacro:door_base_form/>
-    <material>
-      <script>
-          <uri>file://media/materials/scripts/gazebo.material</uri>
-          <name>Gazebo/Yellow</name>
-      </script>
-    </material>
-  </visual>
-  <inertial>
-    <mass>10000</mass>
-  </inertial>
-</link>
-<link name="door">
-  <self_collide>false</self_collide>
-  <pose>0 -1.15 0 0 0 ${-pi/2}</pose>
-  <xacro:macro name="door_form">
-    <geometry>
-      <box><size>1 0.1 1.8</size></box>
-    </geometry>
-  </xacro:macro>
-  <collision name="door_collision">
-    <xacro:door_form/>
-  </collision>
-  <visual name="door_visual">
-    <xacro:door_form/>
-    <material>
-      <script>
-          <uri>file://media/materials/scripts/gazebo.material</uri>
-          <name>Gazebo/Red</name>
-      </script>
-    </material>
-  </visual>
-</link>
+<xacro:cuboid name="door_base" a="4" b="${base_width}" c="2" weight="10000" is_kinematic="true"/>
+<xacro:cuboid name="door" pose="0 -1.15 0 0 0 ${-pi/2}" a="1" b="0.1" c="1.8" weight="5" color="Red"/>
 <joint name="door_to_door_base_joint" type="revolute">
   <parent>door_base</parent>

File: src/simulation/models/worlds/plane.sdf.xacro (robot description, xacro)
@@ -13,8 +13,14 @@
 </model>
 <include>
-    <name>door</name>
-    <uri>file:/$(env MODELS_DIR)/objects/simple_door</uri>
+    <name>switch_wall</name>
+    <uri>file:/$(env MODELS_DIR)/objects/test/switch_with_base</uri>
     <pose>5 0 1 0 0 0</pose>
 </include>
+<include>
+    <name>door</name>
+    <uri>file:/$(env MODELS_DIR)/objects/test/simple_door</uri>
+    <pose>0 5 1 0 0 0</pose>
+</include>
+<!--
 <plugin
     filename="${gazebo_systems_lib_dir}/libDoorButtonSystem.so"
@@ -25,9 +31,4 @@
     <opening_force>20</opening_force>
 </plugin>
-<!--
-<plugin filename="gz-sim-python-system-loader-system" name="gz::sim::systems::PythonSystemLoader">
-    <module_name>systems/door.py</module_name>
-    <force>100</force>
-</plugin>
 -->
 </world>

Commit message: wip

File: src/simulation/models/common/utils.xacro (robot description, xacro)
@@ -8,4 +8,15 @@
       <box><size>${a} ${b} ${c}</size></box>
     </geometry>
+</xacro:macro>
+<xacro:macro name="cuboid_inertia" params="weight a b c pose:='0 0 0 0 0 0'">
+  <inertial>
+    <pose>${pose}</pose>
+    <mass>${weight}</mass>
+    <inertia>
+      <ixx>${weight * (a**2 + c**2) / 12}</ixx>
+      <iyy>${weight * (b**2 + c**2) / 12}</iyy>
+      <izz>${weight * (b**2 + a**2) / 12}</izz>
+    </inertia>
+  </inertial>
 </xacro:macro>
 <xacro:macro name="cuboid" params="name a b c weight pose:='0 0 0 0 0 0' color:=Yellow is_kinematic:=false self_collide:=false">
@@ -26,12 +37,5 @@
     </material>
   </visual>
-  <inertial>
-    <mass>${weight}</mass>
-    <inertia>
-      <ixx>${weight * (a**2 + c**2) / 12}</ixx>
-      <iyy>${weight * (b**2 + c**2) / 12}</iyy>
-      <izz>${weight * (b**2 + a**2) / 12}</izz>
-    </inertia>
-  </inertial>
+  <xacro:cuboid_inertia weight="${weight}" a="${a}" b="${b}" c="${c}"/>
 </link>
 </xacro:macro>

File: src/simulation/models/objects/switch/model.sdf.xacro (robot description, xacro)
@@ -2,58 +2,6 @@
 <sdf xmlns:xacro="http://www.ros.org/wiki/xacro" version="1.10">
 <model name="switch">
-<link name="frame">
-    <xacro:macro name="frame_stl">
-        <geometry>
-          <mesh>
-            <uri>file:/$(env MODELS_DIR)/objects/switch/01_base.stl</uri>
-            <scale>1 1 1</scale>
-          </mesh>
-        </geometry>
-      </xacro:macro>
-      <visual name="frame_visual">
-        <xacro:frame_stl/>
-        <material>
-          <script>
-              <uri>file://media/materials/scripts/gazebo.material</uri>
-              <name>Gazebo/Red</name>
-          </script>
-        </material>
-      </visual>
-</link>
-<link name="tumbler">
-    <pose>0 0 -0.021 0 0 0</pose>
-    <xacro:macro name="tumbler_stl">
-        <geometry>
-          <mesh>
-            <uri>file:/$(env MODELS_DIR)/objects/switch/01_tumbler.stl</uri>
-            <scale>1 1 1</scale>
-          </mesh>
-        </geometry>
-      </xacro:macro>
-      <collision name="tumbler_collision">
-        <xacro:tumbler_stl/>
-      </collision>
-      <visual name="tumbler_visual">
-        <xacro:tumbler_stl/>
-        <material>
-          <script>
-              <uri>file://media/materials/scripts/gazebo.material</uri>
-              <name>Gazebo/Red</name>
-          </script>
-        </material>
-      </visual>
-</link>
-<joint name="tumbler_to_frame_joint" type="revolute">
-    <parent>frame</parent>
-    <child>tumbler</child>
-    <pose>0 0 0 0 0 0</pose>
-    <axis>
-      <xyz>0 1 0</xyz>
-      <limit>
-        <lower>${-pi/4}</lower>
-        <upper>${+pi/4}</upper>
-      </limit>
-    </axis>
-</joint>
+<xacro:include filename="switch.xacro" />
+<xacro:switch/>
 </model>
 </sdf>

File: src/simulation/models/objects/switch_rotate/model.sdf.xacro (robot description, xacro)
@@ -3,4 +3,5 @@
 <model name="rotating_switch">
 <link name="frame">
+  <self_collide>false</self_collide>
   <visual name="frame_visual">
     <geometry>
@@ -19,4 +20,5 @@
 </link>
 <link name="rotator">
+    <self_collide>false</self_collide>
     <pose>0 0 -0.004 0 0 0</pose>
     <xacro:macro name="rotator_stl">

File: src/simulation/models/worlds/plane.sdf.xacro (robot description, xacro)
@@ -36,4 +36,13 @@
     <is_oneshot>true</is_oneshot>
 </plugin>
+<!-- TESTS -->
+<include>
+    <uri>file:/$(env MODELS_DIR)/objects/garage-inter</uri>
+    <pose>-5 0 0 0 0 0</pose>
+</include>
+<joint name="garage_to_world" type="fixed">
+    <parent>world</parent>
+    <child>garage::garage</child>
+</joint>
 </world>
 </sdf>
