Commit message: add camera to ruka and update colors

File: src/simulation/models/common/plugins.xacro (robot description, xacro)
@@ -12,6 +12,6 @@
     name="gz::sim::systems::SceneBroadcaster">
 </plugin>
-<physics name="1ms" type="ignored">
-    <max_step_size>0.001</max_step_size>
+<physics name="10ms" type="ignored">
+    <max_step_size>0.01</max_step_size>
     <real_time_factor>1.0</real_time_factor>
 </physics>
@@ -21,5 +21,5 @@
 <plugin filename="gz-sim-sensors-system"
         name="gz::sim::systems::Sensors">
-    <render_engine>ogre2</render_engine>
+    <render_engine>ogre</render_engine>
 </plugin>
 </include>

File: src/simulation/models/explorer/explorer.urdf.xacro (robot description, xacro)
@@ -3,9 +3,30 @@
 <xacro:include filename="$(env MODELS_DIR)/rover/rover.urdf.xacro" />
 <xacro:include filename="$(find ruka_gz)/config/ruka_gz.urdf.xacro" />
-<xacro:include filename="$(env MODELS_DIR)/objects/cameras/d435.xacro" />
+<xacro:include filename="$(env MODELS_DIR)/objects/cameras/d405.xacro" />
 <joint name="ruka_to_rover" type="fixed">
     <parent link="base"/>
     <child link="base_link"/>
     <origin rpy="0 0 0" xyz="0.2 0 0.251"/>
+</joint>
+<link name="ruka_realsense_mount">
+    <visual name="ruka_realsense_mount_visual">
+        <geometry>
+            <mesh filename="file://$(env MODELS_DIR)/explorer/j5-d405-mount.stl"/>
+        </geometry>
+        <material name="black">
+            <color rgba="0 0 0 1.0"/>
+        </material>
+    </visual>
+</link>
+<joint name="realsense_mount_to_ruka" type="fixed">
+    <parent link="link_05"/>
+    <child link="ruka_realsense_mount"/>
+    <origin xyz="0.029 -0.009 0" rpy="${pi/2} -${pi/2} ${pi/2}"/>
+</joint>
+<xacro:realsense-d405 suffix='_ruka'/>
+<joint name="camera_to_ruka" type="fixed">
+    <parent link="ruka_realsense_mount"/>
+    <child link="realsense_d405_ruka_frame"/>
+    <origin xyz="0 0.014 0.058" rpy="0 0.35 ${pi/2}" />
 </joint>
 <gazebo>

File: src/simulation/models/objects/01-module/module.xacro (robot description, xacro)
@@ -22,5 +22,5 @@
             <script>
                 <uri>file://media/materials/scripts/gazebo.material</uri>
-                <name>Gazebo/Yellow</name>
+                <name>Gazebo/White</name>
             </script>
         </material>

File: src/simulation/models/objects/button/button.xacro (robot description, xacro)
@@ -16,5 +16,5 @@
           <script>
               <uri>file://media/materials/scripts/gazebo.material</uri>
-              <name>Gazebo/Red</name>
+              <name>Gazebo/Gray</name>
           </script>
         </material>

File: src/simulation/models/objects/cameras/d405.xacro (robot description, xacro)
@@ -15,5 +15,5 @@
     <parent link="realsense_d405${suffix}_frame"/>
     <child link="realsense_d405${suffix}_camera"/>
-    <origin xyz="0.024 0 0" rpy="${pi/2} 0 0"/>
+    <origin xyz="0.024 0 0.024" rpy="0 0 0"/>
 </joint>
 <gazebo reference="realsense_d405${suffix}_camera">
@@ -26,5 +26,5 @@
             </image>
             <clip>
-                <near>0.1</near>
+                <near>0.01</near>
                 <far>100</far>
             </clip>

File: src/simulation/models/objects/garage/model.sdf.xacro (robot description, xacro)
@@ -23,5 +23,5 @@
             <script>
                 <uri>file://media/materials/scripts/gazebo.material</uri>
-                <name>Gazebo/Yellow</name>
+                <name>Gazebo/White</name>
             </script>
         </material>
@@ -48,5 +48,5 @@
             <script>
                 <uri>file://media/materials/scripts/gazebo.material</uri>
-                <name>Gazebo/Red</name>
+                <name>Gazebo/Blue</name>
             </script>
         </material>

File: src/simulation/models/objects/main-panel/main-panel.xacro (robot description, xacro)
@@ -21,5 +21,5 @@
             <script>
                 <uri>file://media/materials/scripts/gazebo.material</uri>
-                <name>Gazebo/Yellow</name>
+                <name>Gazebo/White</name>
             </script>
         </material>

File: src/simulation/models/objects/marker/marker.xacro (robot description, xacro)
@@ -21,5 +21,5 @@
       <script>
         <uri>file://media/materials/scripts/gazebo.material</uri>
-        <name>Gazebo/Yellow</name>
+        <name>Gazebo/White</name>
       </script>
     </material>

File: src/simulation/models/objects/switch/switch.xacro (robot description, xacro)
@@ -16,5 +16,5 @@
           <script>
               <uri>file://media/materials/scripts/gazebo.material</uri>
-              <name>Gazebo/Red</name>
+              <name>Gazebo/Gray</name>
           </script>
         </material>

File: src/simulation/models/objects/switch_room/switch_room.xacro (robot description, xacro)
@@ -16,5 +16,5 @@
           <script>
               <uri>file://media/materials/scripts/gazebo.material</uri>
-              <name>Gazebo/Red</name>
+              <name>Gazebo/White</name>
           </script>
         </material>
@@ -40,5 +40,5 @@
           <script>
               <uri>file://media/materials/scripts/gazebo.material</uri>
-              <name>Gazebo/Red</name>
+              <name>Gazebo/White</name>
           </script>
         </material>

File: src/simulation/models/objects/switch_rotate/rotator.xacro (robot description, xacro)
@@ -13,5 +13,5 @@
         <script>
           <uri>file://media/materials/scripts/gazebo.material</uri>
-          <name>Gazebo/Red</name>
+          <name>Gazebo/Gray</name>
         </script>
       </material>

File: src/simulation/models/objects/weight-button/weight_button.xacro (robot description, xacro)
@@ -16,5 +16,5 @@
           <script>
               <uri>file://media/materials/scripts/gazebo.material</uri>
-              <name>Gazebo/Red</name>
+              <name>Gazebo/Gray</name>
           </script>
         </material>
@@ -40,5 +40,5 @@
           <script>
               <uri>file://media/materials/scripts/gazebo.material</uri>
-              <name>Gazebo/Red</name>
+              <name>Gazebo/Blue</name>
           </script>
         </material>
