Commit message: garage

File: src/simulation/models/objects/garage-inter/model.sdf.xacro (robot description, xacro)
@@ -54,13 +54,30 @@
     <xacro:cuboid_inertia weight="5" a="0.2" b="0.7" c="2"/>
 </link>
-<joint name="garage_door_joint" type="fixed">
+<joint name="garage_door_joint" type="prismatic">
     <parent>garage</parent>
     <child>door</child>
+    <axis>
+        <xyz>1 0 0</xyz>
+        <limit>
+            <lower>0</lower>
+            <upper>1</upper>
+        </limit>
+        <dynamics>
+            <damping>0</damping>
+            <spring_stiffness>0</spring_stiffness>
+            <spring_reference>0</spring_reference>
+        </dynamics>
+    </axis>
+    <physics>
+        <ode>
+            <cfm_damping>1</cfm_damping>
+        </ode>
+    </physics>
 </joint>
-<xacro:include filename="$(env MODELS_DIR)/objects/switch/switch.xacro" />
+<xacro:include filename="$(env MODELS_DIR)/objects/button/button.xacro" />
 <xacro:macro name="garage_button" params="name pose">
     <model name="${name}_button">
         <pose>${pose}</pose>
-        <xacro:switch name_prefix="${name}_"/>
+        <xacro:button name_prefix="${name}_"/>
     </model>
     <joint name="${name}_button_to_wall_joint" type="fixed">
@@ -69,8 +86,8 @@
     </joint>
 </xacro:macro>
-<xacro:garage_button name="outer_open" pose="1.65 0 0.85 ${-pi/2} 0 0"/>
-<xacro:garage_button name="outer_close" pose="1.65 0 0.7 ${-pi/2} 0 0"/>
-<xacro:garage_button name="inner_open" pose="0.1 0.4 0.9 0 ${-pi/2} ${-pi/2}"/>
-<xacro:garage_button name="inner_close" pose="0.1 0.4 0.7 0 ${-pi/2} ${-pi/2}"/>
+<xacro:garage_button name="outer_open" pose="1.65 0 0.85 ${-pi/2} 0 ${pi}"/>
+<xacro:garage_button name="outer_close" pose="1.65 0 0.7 ${-pi/2} 0 ${pi}"/>
+<xacro:garage_button name="inner_open" pose="0.1 0.4 0.9 0 ${-pi/2} ${pi}"/>
+<xacro:garage_button name="inner_close" pose="0.1 0.4 0.7 0 ${-pi/2} ${pi}"/>
 </model>
 </sdf>

File: src/simulation/models/worlds/plane.sdf.xacro (robot description, xacro)
@@ -27,14 +27,4 @@
     <pose>0 -5 1 0 0 0</pose>
 </include>
-<plugin
-    filename="${gazebo_systems_lib_dir}/libTriggerSystems.so"
-    name="trigger_systems::DoorButton">
-    <hinge_joint>door_to_door_base_joint</hinge_joint>
-    <trigger_joint>button_to_door_base_joint</trigger_joint>
-    <percentage_activated>50</percentage_activated>
-    <opening_force>800</opening_force>
-    <is_oneshot>true</is_oneshot>
-</plugin>
-<!-- TESTS -->
 <include>
     <uri>file:/$(env MODELS_DIR)/objects/garage-inter</uri>
@@ -45,4 +35,24 @@
     <child>garage::garage</child>
 </joint>
+<xacro:macro
+    name="garage_door_trigger"
+    params="name force"
+>
+    <plugin
+        filename="${gazebo_systems_lib_dir}/libTriggerSystems.so"
+        name="trigger_systems::DoorButton">
+        <hinge_joint>garage_door_joint</hinge_joint>
+        <trigger_joint>${name}_button_to_frame_joint</trigger_joint>
+        <percentage_activated>50</percentage_activated>
+        <opening_force>${force}</opening_force>
+        <closing_force>0</closing_force>
+        <is_oneshot>true</is_oneshot>
+        <log_name>${name}</log_name>
+    </plugin>
+</xacro:macro>
+<xacro:garage_door_trigger name="outer_open" force="5000"/>
+<xacro:garage_door_trigger name="outer_close" force="-5000"/>
+<xacro:garage_door_trigger name="inner_open" force="5000"/>
+<xacro:garage_door_trigger name="inner_close" force="-5000"/>
 </world>
 </sdf>
