Commit message: base-panel

File: src/simulation/models/objects/garage/model.sdf.xacro (robot description, xacro)
@@ -1,29 +1,93 @@
 <?xml version="1.0" ?>
 <sdf xmlns:xacro="http://www.ros.org/wiki/xacro" version="1.10">
-  <model name="garage">
-    <pose>0 0 0 0 0 0</pose>
-    <static>true</static>
-    <link name="garage">
-      <xacro:macro name="garage_stl">
+<model name="garage">
+<pose>0 0 0 0 0 0</pose>
+<static>false</static>
+<xacro:include filename="$(env MODELS_DIR)/common/utils.xacro" />
+<link name="garage">
+    <self_collide>false</self_collide>
+    <xacro:macro name="garage_stl">
         <geometry>
-          <mesh>
-            <uri>file:/$(env MODELS_DIR)/objects/garage/base1.stl</uri>
-            <scale>1 1 1</scale>
-          </mesh>
+            <mesh>
+                <uri>file:/$(env MODELS_DIR)/objects/garage/base1-asm.stl</uri>
+                <scale>1 1 1</scale>
+            </mesh>
         </geometry>
-      </xacro:macro>
-      <collision name="garage_collision">
+    </xacro:macro>
+    <collision name="garage_collision">
         <xacro:garage_stl/>
-      </collision>
-      <visual name="garage_visual">
+    </collision>
+    <visual name="garage_visual">
         <xacro:garage_stl/>
         <material>
-          <script>
-              <uri>file://media/materials/scripts/gazebo.material</uri>
-              <name>Gazebo/Red</name>
-          </script>
+            <script>
+                <uri>file://media/materials/scripts/gazebo.material</uri>
+                <name>Gazebo/Yellow</name>
+            </script>
         </material>
-      </visual>
-    </link>
-  </model>
+    </visual>
+    <xacro:cuboid_inertia pose="2 1 1 0 0 0" weight="10000" a="4" b="2" c="2"/>
+</link>
+<link name="door">
+    <self_collide>false</self_collide>
+    <pose>0.4 0.05 0.1 0 0 0</pose>
+    <xacro:macro name="door_stl">
+        <geometry>
+            <mesh>
+            <uri>file:/$(env MODELS_DIR)/objects/garage/base-door.stl</uri>
+            <scale>1 1 1</scale>
+            </mesh>
+        </geometry>
+    </xacro:macro>
+    <collision name="garage_collision">
+        <xacro:door_stl/>
+    </collision>
+    <visual name="garage_visual">
+        <xacro:door_stl/>
+        <material>
+            <script>
+                <uri>file://media/materials/scripts/gazebo.material</uri>
+                <name>Gazebo/Red</name>
+            </script>
+        </material>
+    </visual>
+    <xacro:cuboid_inertia weight="5" a="0.2" b="0.7" c="2"/>
+</link>
+<joint name="garage_door_joint" type="prismatic">
+    <parent>garage</parent>
+    <child>door</child>
+    <axis>
+        <xyz>1 0 0</xyz>
+        <limit>
+            <lower>0</lower>
+            <upper>1</upper>
+        </limit>
+        <dynamics>
+            <damping>0</damping>
+            <spring_stiffness>0</spring_stiffness>
+            <spring_reference>0</spring_reference>
+        </dynamics>
+    </axis>
+    <physics>
+        <ode>
+            <cfm_damping>1</cfm_damping>
+        </ode>
+    </physics>
+</joint>
+<xacro:include filename="$(env MODELS_DIR)/objects/button/button.xacro" />
+<xacro:macro name="garage_button" params="name pose">
+    <model name="${name}_button">
+        <pose>${pose}</pose>
+        <xacro:button name_prefix="${name}_"/>
+    </model>
+    <joint name="${name}_button_to_wall_joint" type="fixed">
+        <parent>garage</parent>
+        <child>${name}_button::${name}_frame</child>
+    </joint>
+</xacro:macro>
+<xacro:garage_button name="outer_open" pose="1.65 0 0.85 ${-pi/2} 0 ${pi}"/>
+<xacro:garage_button name="outer_close" pose="1.65 0 0.7 ${-pi/2} 0 ${pi}"/>
+<xacro:garage_button name="inner_open" pose="0.1 0.4 0.9 0 ${-pi/2} ${pi}"/>
+<xacro:garage_button name="inner_close" pose="0.1 0.4 0.7 0 ${-pi/2} ${pi}"/>
+</model>
 </sdf>

File: src/simulation/models/objects/switch_rotate/model.sdf.xacro (robot description, xacro)
@@ -2,57 +2,6 @@
 <sdf xmlns:xacro="http://www.ros.org/wiki/xacro" version="1.10">
 <model name="rotating_switch">
-<link name="frame">
-  <self_collide>false</self_collide>
-  <visual name="frame_visual">
-    <geometry>
-      <mesh>
-        <uri>file:/$(env MODELS_DIR)/objects/switch_rotate/02-rotsw-base.stl</uri>
-        <scale>1 1 1</scale>
-      </mesh>
-    </geometry>
-    <material>
-      <script>
-        <uri>file://media/materials/scripts/gazebo.material</uri>
-        <name>Gazebo/Red</name>
-      </script>
-    </material>
-  </visual>
-</link>
-<link name="rotator">
-    <self_collide>false</self_collide>
-    <pose>0 0 -0.004 0 0 0</pose>
-    <xacro:macro name="rotator_stl">
-        <geometry>
-          <mesh>
-            <uri>file:/$(env MODELS_DIR)/objects/switch_rotate/02-rotate-switch.stl</uri>
-            <scale>1 1 1</scale>
-          </mesh>
-        </geometry>
-      </xacro:macro>
-      <collision name="rotator_collision">
-        <xacro:rotator_stl/>
-      </collision>
-      <visual name="rotator_visual">
-        <xacro:rotator_stl/>
-        <material>
-          <script>
-              <uri>file://media/materials/scripts/gazebo.material</uri>
-              <name>Gazebo/Red</name>
-          </script>
-        </material>
-      </visual>
-</link>
-<joint name="rotator_to_frame_joint" type="revolute">
-    <parent>frame</parent>
-    <child>rotator</child>
-    <pose>0 0 0 0 0 0</pose>
-    <axis>
-      <xyz>0 0 1</xyz>
-      <limit>
-        <lower>${-pi}</lower>
-        <upper>${+pi}</upper>
-      </limit>
-    </axis>
-</joint>
+<xacro:include filename="rotator.xacro" />
+<xacro:rotator/>
 </model>
 </sdf>

File: src/simulation/models/worlds/plane.sdf.xacro (robot description, xacro)
@@ -13,21 +13,6 @@
 </model>
 <include>
-    <name>switch_wall</name>
-    <uri>file:/$(env MODELS_DIR)/objects/test/switch_with_base</uri>
-    <pose>5 0 1 0 0 0</pose>
-</include>
-<include>
-    <name>door</name>
-    <uri>file:/$(env MODELS_DIR)/objects/test/simple_door</uri>
-    <pose>0 5 1 0 0 0</pose>
-</include>
-<include>
-    <name>rotator_wall</name>
-    <uri>file:/$(env MODELS_DIR)/objects/test/rotator_with_base</uri>
-    <pose>0 -5 1 0 0 0</pose>
-</include>
-<include>
-    <uri>file:/$(env MODELS_DIR)/objects/garage-inter</uri>
-    <pose>-5 0 0 0 0 0</pose>
+    <uri>file:/$(env MODELS_DIR)/objects/garage</uri>
+    <pose>5 0 0 0 0 0</pose>
 </include>
 <joint name="garage_to_world" type="fixed">
@@ -35,8 +20,5 @@
     <child>garage::garage</child>
 </joint>
-<xacro:macro
-    name="garage_door_trigger"
-    params="name force"
->
+<xacro:macro name="garage_door_trigger" params="name force">
     <plugin
         filename="${gazebo_systems_lib_dir}/libTriggerSystems.so"
@@ -55,4 +37,12 @@
 <xacro:garage_door_trigger name="inner_open" force="5000"/>
 <xacro:garage_door_trigger name="inner_close" force="-5000"/>
+<include>
+    <uri>file:/$(env MODELS_DIR)/objects/main-panel</uri>
+    <pose>-5 0 2 0 0 0</pose>
+</include>
+<joint name="panel_to_world" type="fixed">
+    <parent>world</parent>
+    <child>main-panel::panel</child>
+</joint>
 </world>
 </sdf>
