Commit message: working panel

File: src/simulation/models/objects/button/button.xacro (robot description, xacro)
@@ -31,9 +31,9 @@
           </mesh>
         </geometry>
-      </xacro:macro>
-      <collision name="button_collision">
+    </xacro:macro>
+    <collision name="button_collision">
         <xacro:button_stl/>
-      </collision>
-      <visual name="button_visual">
+    </collision>
+    <visual name="button_visual">
         <xacro:button_stl/>
         <material>
@@ -43,5 +43,5 @@
           </script>
         </material>
-      </visual>
+    </visual>
 </link>
 <joint name="${name_prefix}button_to_frame_joint" type="prismatic">

File: src/simulation/models/objects/main-panel/model.sdf.xacro (robot description, xacro)
@@ -53,4 +53,49 @@
     <child>panel_image</child>
 </joint>
+<link name="panel_door">
+    <pose>0.46 0.16 -0.008 0 0 0</pose>
+    <self_collide>false</self_collide>
+    <xacro:macro name="panel_door_stl">
+        <geometry>
+            <mesh>
+                <uri>file:/$(env MODELS_DIR)/objects/main-panel/sampler-door.stl</uri>
+                <scale>1 1 1</scale>
+            </mesh>
+        </geometry>
+    </xacro:macro>
+    <collision name="panel_door_collision">
+        <xacro:panel_door_stl/>
+    </collision>
+    <visual name="panel_door_visual">
+        <xacro:panel_door_stl/>
+        <material>
+            <script>
+                <uri>file://media/materials/scripts/gazebo.material</uri>
+                <name>Gazebo/Blue</name>
+            </script>
+        </material>
+    </visual>
+</link>
+<joint name="panel_door_joint" type="prismatic">
+    <parent>panel</parent>
+    <child>panel_door</child>
+    <axis>
+        <xyz>-1 0 0</xyz>
+        <limit>
+            <lower>0</lower>
+            <upper>0.18</upper>
+        </limit>
+        <dynamics>
+            <damping>0</damping>
+            <spring_stiffness>0</spring_stiffness>
+            <spring_reference>0</spring_reference>
+        </dynamics>
+    </axis>
+    <physics>
+        <ode>
+            <cfm_damping>1</cfm_damping>
+        </ode>
+    </physics>
+</joint>
 <xacro:include filename="$(env MODELS_DIR)/objects/switch_rotate/rotator.xacro" />
 <xacro:include filename="$(env MODELS_DIR)/objects/switch/switch.xacro" />
@@ -83,5 +128,5 @@
 </xacro:macro>
 <xacro:trigger type="rotator" name="door_rotator" pose="0.53 0.095 0 0 0 0"/>
-<xacro:trigger type="weight_button" name="secret-button" pose="0.55 0.16 -0.06 ${pi/2} 0 0"/>
+<xacro:trigger type="weight_button" name="secret-button" pose="0.55 0.16 -0.06 ${-pi/2} 0 0"/>
 <xacro:trigger type="switch_room" name="switch_room" pose="0.16 0.29 0 0 0 ${-pi/2}"/>
 <xacro:trigger type="button" name="button-1" pose="0.291 0.289 0 0 0 0"/>

File: src/simulation/models/objects/switch_rotate/rotator.xacro (robot description, xacro)
@@ -49,5 +49,5 @@
         <xyz>0 0 1</xyz>
         <limit>
-            <lower>${-pi}</lower>
+            <lower>0</lower>
             <upper>${+pi}</upper>
         </limit>

File: src/simulation/models/worlds/plane.sdf.xacro (robot description, xacro)
@@ -31,4 +31,5 @@
         <is_oneshot>true</is_oneshot>
         <log_name>${name}</log_name>
+        <do_log>false</do_log>
     </plugin>
 </xacro:macro>
@@ -45,4 +46,16 @@
     <child>main-panel::panel</child>
 </joint>
+<plugin
+    filename="${gazebo_systems_lib_dir}/libTriggerSystems.so"
+    name="trigger_systems::DoorButton">
+    <hinge_joint>panel_door_joint</hinge_joint>
+    <trigger_joint>door_rotator_rotator_to_frame_joint</trigger_joint>
+    <percentage_activated>50</percentage_activated>
+    <opening_force>100</opening_force>
+    <closing_force>-100</closing_force>
+    <is_oneshot>true</is_oneshot>
+    <log_name>panel_door</log_name>
+    <do_log>true</do_log>
+</plugin>
 </world>
 </sdf>
