Commit message: simple sim

File: src/simulation/models/rover/rover.xacro (robot description, xacro)
@@ -40,4 +40,42 @@
     <child link="base_weight"/>
 </joint>
+<!-- CAMERA BLOCK-->
+<link name="camera"></link>
+<joint name="camera_joint" type="fixed">
+    <parent link="base"/>
+    <child link="camera"/>
+    <origin xyz="0 0 ${robot_side_len/2}"/>
+</joint>
+<gazebo reference="camera">
+    <sensor name="camera" type="camera">
+        <camera>
+            <horizontal_fov>1.047</horizontal_fov>
+            <image>
+                <width>320</width>
+                <height>240</height>
+            </image>
+            <clip>
+                <near>0.1</near>
+                <far>100</far>
+            </clip>
+        </camera>
+        <always_on>1</always_on>
+        <update_rate>30</update_rate>
+        <visualize>true</visualize>
+        <topic>camera</topic>
+    </sensor>
+</gazebo>
+<!-- END CAMERA BLOCK-->
+<gazebo>
+    <plugin
+        filename="gz-sim-odometry-publisher-system"
+        name="gz::sim::systems::OdometryPublisher">
+        <odom_frame>odom</odom_frame>
+        <robot_base_frame>base</robot_base_frame>
+        <odom_publish_frequency>20</odom_publish_frequency>
+        <odom_topic>odom</odom_topic>
+        <tf_topic>tf</tf_topic>
+  </plugin>
+</gazebo>
 </xacro:macro>
 </include>

Commit message: update rover model

File: src/simulation/models/rover/rover.xacro (robot description, xacro)
@@ -4,11 +4,16 @@
 <xacro:include filename="sslidar.xacro" />
 <xacro:include filename="wheel.xacro" />
-<xacro:property name="robot_side_len" value="0.2" />
+<xacro:property name="robot_side_x" value="0.7" />
+<xacro:property name="robot_side_y" value="0.7" />
+<xacro:property name="robot_side_z" value="0.5" />
 <xacro:property name="robot_mass" value="2" />
+<xacro:property name="wheel_x_offset" value="0.4" />
+<xacro:property name="wheel_y_offset" value="0.4" />
+<xacro:property name="wheel_diameter" value="0.3" />
 <link name="base">
     <visual name="base_visual">
         <origin  xyz="0 0 0" rpy="0 0 0"/>
         <geometry>
-            <box size="${robot_side_len} ${robot_side_len} ${robot_side_len}" />
+            <box size="${robot_side_x} ${robot_side_y} ${robot_side_z}" />
         </geometry>
         <material name="blue">
@@ -19,5 +24,5 @@
         <origin  xyz="0 0 0"/>
         <geometry>
-            <box size="${robot_side_len} ${robot_side_len} ${robot_side_len}" />
+            <box size="${robot_side_x} ${robot_side_y} ${robot_side_z}" />
         </geometry>
     </collision>
@@ -30,5 +35,5 @@
     <visual name="base_visual">
         <geometry>
-            <sphere radius="${robot_side_len / 2 + 0.025}"/>
+            <sphere radius="${robot_side_z / 2 + 0.025}"/>
             <material name="red">
                 <color rgba="1.0 0 0 1.0"/>
@@ -41,8 +46,8 @@
     <child link="base_weight"/>
 </joint>
-<xacro:wheel index="0" xyz="1 -1 0" axis="0 0 -1"/>
-<xacro:wheel index="1" xyz="-1 -1 0" axis="0 0 -1"/>
-<xacro:wheel index="2" xyz="1 1 0" axis="0 0 -1"/>
-<xacro:wheel index="3" xyz="-1 1 0" axis="0 0 -1"/>
+<xacro:wheel index="0" xyz="${wheel_x_offset} ${-wheel_y_offset} 0" axis="0 0 -1" diameter="${wheel_diameter}"/>
+<xacro:wheel index="1" xyz="${-wheel_x_offset} ${-wheel_y_offset} 0" axis="0 0 -1" diameter="${wheel_diameter}"/>
+<xacro:wheel index="2" xyz="${wheel_x_offset} ${wheel_y_offset} 0" axis="0 0 -1" diameter="${wheel_diameter}"/>
+<xacro:wheel index="3" xyz="${-wheel_x_offset} ${wheel_y_offset} 0" axis="0 0 -1" diameter="${wheel_diameter}"/>
 <!-- CAMERA BLOCK-->
 <link name="camera"></link>
@@ -50,5 +55,5 @@
     <parent link="base"/>
     <child link="camera"/>
-    <origin xyz="0 0 ${robot_side_len/2}"/>
+    <origin xyz="0 0 ${robot_side_z/2}"/>
 </joint>
 <gazebo reference="camera">
@@ -102,6 +107,6 @@
         <right_joint>wheel_3_joint</right_joint>
         <!-- kinematics -->
-        <wheel_separation>2.0</wheel_separation>
-        <wheel_diameter>0.4</wheel_diameter>
+        <wheel_separation>${wheel_y_offset*2}</wheel_separation>
+        <wheel_diameter>${wheel_diameter}</wheel_diameter>
         <!-- ODOMETRY -->
         <odom_publish_frequency>0</odom_publish_frequency>

File: src/simulation/models/rover/wheel.xacro (robot description, xacro)
@@ -1,4 +1,4 @@
 <include xmlns:xacro="http://www.ros.org/wiki/xacro">
-<xacro:macro name="wheel" params="index xyz axis">
+<xacro:macro name="wheel" params="index xyz axis diameter">
 <link name="wheel_${index}">
     <inertial>
@@ -8,10 +8,10 @@
     <visual name="wheel_${index}_visual">
         <geometry>
-            <cylinder radius="0.4" length="0.2"/>
+            <cylinder radius="${diameter}" length="0.1"/>
         </geometry>
     </visual>
     <collision name='wheel_${index}_collision'>
         <geometry>
-            <cylinder radius="0.4" length="0.2"/>
+            <cylinder radius="${diameter}" length="0.1"/>
         </geometry>
     </collision>

File: src/simulation/models/worlds/field/field.sdf.xacro (robot description, xacro)
@@ -18,4 +18,8 @@
     <pose>0 5 1 0 0 0</pose>
 </include>
+<include>
+    <uri>file:/$(env MODELS_DIR)/objects/garage</uri>
+    <pose>0 -8 0 0 0 ${pi}</pose>
+</include>
 <model name='rover'>
     <include>

Commit message: add rover model

File: src/simulation/models/rover/rover.xacro (robot description, xacro)
@@ -4,23 +4,28 @@
 <xacro:include filename="sslidar.xacro" />
 <xacro:include filename="wheel.xacro" />
-<xacro:property name="robot_side_x" value="0.7" />
-<xacro:property name="robot_side_y" value="0.7" />
-<xacro:property name="robot_side_z" value="0.5" />
-<xacro:property name="robot_mass" value="2" />
-<xacro:property name="wheel_x_offset" value="0.4" />
-<xacro:property name="wheel_y_offset" value="0.4" />
-<xacro:property name="wheel_diameter" value="0.3" />
+<xacro:property name="robot_side_x" value="0.898" />
+<xacro:property name="robot_side_y" value="0.426" />
+<xacro:property name="robot_side_z" value="0.278" />
+<xacro:property name="z_offset_to_center" value="${robot_side_z / 2 - 0.043}" />
+<xacro:property name="robot_mass" value="30" />
+<xacro:property name="wheel_x_offset" value="0.25" />
+<xacro:property name="wheel_y_offset" value="0.3005" />
+<xacro:property name="wheel_radius" value="0.185" />
 <link name="base">
     <visual name="base_visual">
-        <origin  xyz="0 0 0" rpy="0 0 0"/>
         <geometry>
-            <box size="${robot_side_x} ${robot_side_y} ${robot_side_z}" />
+            <mesh filename="file://$(env MODELS_DIR)/rover/stl/explorer-base.stl"/>
         </geometry>
+        <material name="gray">
+            <color rgba="0.4 0.4 0.4 1.0"/>
+        </material>
+        <!--
         <material name="blue">
             <color rgba="0 0 0.7 1.0"/>
         </material>
+        -->
     </visual>
     <collision name="base_collision">
-        <origin  xyz="0 0 0"/>
+        <origin  xyz="0 0 ${z_offset_to_center}"/>
         <geometry>
             <box size="${robot_side_x} ${robot_side_y} ${robot_side_z}" />
@@ -35,9 +40,10 @@
     <visual name="base_visual">
         <geometry>
-            <sphere radius="${robot_side_z / 2 + 0.025}"/>
-            <material name="red">
-                <color rgba="1.0 0 0 1.0"/>
-            </material>
+            <!--<sphere radius="${robot_side_z / 2 + 0.025}"/>-->
+            <sphere radius="0.1"/>
         </geometry>
+        <material name="blue">
+            <color rgba="0 0 1.0 1.0"/>
+        </material>
     </visual>
 </link>
@@ -45,9 +51,70 @@
     <parent link="base"/>
     <child link="base_weight"/>
+    <origin xyz="0 0 ${z_offset_to_center}" rpy="0 0 0"/>
 </joint>
-<xacro:wheel index="0" xyz="${wheel_x_offset} ${-wheel_y_offset} 0" axis="0 0 -1" diameter="${wheel_diameter}"/>
-<xacro:wheel index="1" xyz="${-wheel_x_offset} ${-wheel_y_offset} 0" axis="0 0 -1" diameter="${wheel_diameter}"/>
-<xacro:wheel index="2" xyz="${wheel_x_offset} ${wheel_y_offset} 0" axis="0 0 -1" diameter="${wheel_diameter}"/>
-<xacro:wheel index="3" xyz="${-wheel_x_offset} ${wheel_y_offset} 0" axis="0 0 -1" diameter="${wheel_diameter}"/>
+<link name="top_face">
+    <visual name="top_face_visual">
+        <geometry>
+            <mesh filename="file://$(env MODELS_DIR)/rover/stl/top-face.stl"/>
+        </geometry>
+        <material name="red">
+            <color rgba="1.0 0 0 1.0"/>
+        </material>
+    </visual>
+</link>
+<link name="top_rails">
+    <visual name="top_rails_visual">
+        <geometry>
+            <mesh filename="file://$(env MODELS_DIR)/rover/stl/top-rails.stl"/>
+        </geometry>
+        <material name="black">
+            <color rgba="0 0 0 1.0"/>
+        </material>
+    </visual>
+</link>
+<link name="bumper_front">
+    <visual name="bumper_front_visual">
+        <geometry>
+            <mesh filename="file://$(env MODELS_DIR)/rover/stl/bumper.stl"/>
+        </geometry>
+        <material name="black">
+            <color rgba="0 0 0 1.0"/>
+        </material>
+    </visual>
+</link>
+<link name="bumper_back">
+    <visual name="bumper_back_visual">
+        <geometry>
+            <mesh filename="file://$(env MODELS_DIR)/rover/stl/bumper.stl"/>
+        </geometry>
+        <material name="black">
+            <color rgba="0 0 0 1.0"/>
+        </material>
+    </visual>
+</link>
+<joint name="bumper_front_to_base" type="fixed">
+    <parent link="base"/>
+    <child link="bumper_front"/>
+    <origin xyz="0.383 0.001 0.029" rpy="${-pi/2} 0 ${-pi/2}"/>
+</joint>
+<joint name="bumper_back_to_base" type="fixed">
+    <parent link="base"/>
+    <child link="bumper_back"/>
+    <origin xyz="-0.383 0.001 0.031" rpy="${pi/2} 0 ${-pi/2}"/>
+</joint>
+<joint name="top_rails_to_base" type="fixed">
+    <parent link="base"/>
+    <child link="top_rails"/>
+    <origin xyz="0 0 0.215" rpy="0 0 0"/>
+</joint>
+<joint name="top_face_to_base" type="fixed">
+    <parent link="base"/>
+    <child link="top_face"/>
+    <origin xyz="0 0 0.213" rpy="0 0 0"/>
+</joint>
+<xacro:wheel index="0" xyz="${wheel_x_offset} ${-wheel_y_offset} 0" yaw="0" axis="0 0 -1" radius="${wheel_radius}"/>
+<xacro:wheel index="1" xyz="${-wheel_x_offset} ${-wheel_y_offset} 0" yaw="0" axis="0 0 -1" radius="${wheel_radius}"/>
+<xacro:wheel index="2" xyz="${wheel_x_offset} ${wheel_y_offset} 0" yaw="${pi}" axis="0 0 1" radius="${wheel_radius}"/>
+<xacro:wheel index="3" xyz="${-wheel_x_offset} ${wheel_y_offset} 0" yaw="${pi}" axis="0 0 1" radius="${wheel_radius}"/>
 <!-- CAMERA BLOCK-->
 <link name="camera"></link>
@@ -108,5 +175,5 @@
         <!-- kinematics -->
         <wheel_separation>${wheel_y_offset*2}</wheel_separation>
-        <wheel_diameter>${wheel_diameter}</wheel_diameter>
+        <wheel_diameter>${wheel_radius * 2}</wheel_diameter>
         <!-- ODOMETRY -->
         <odom_publish_frequency>0</odom_publish_frequency>

File: src/simulation/models/rover/wheel.xacro (robot description, xacro)
@@ -1,24 +1,41 @@
 <include xmlns:xacro="http://www.ros.org/wiki/xacro">
-<xacro:macro name="wheel" params="index xyz axis diameter">
-<link name="wheel_${index}">
+<xacro:macro name="wheel" params="index xyz yaw axis radius">
+<link name="wheel_${index}_disc">
     <inertial>
         <mass value="1"/>
         <inertia ixx="0.043333" ixy="0" ixz="0" iyy="0.043333" iyz="0" izz="0.08"/>
     </inertial>
-    <visual name="wheel_${index}_visual">
+    <visual name="wheel_${index}_disc_visual">
         <geometry>
-            <cylinder radius="${diameter}" length="0.1"/>
+            <mesh filename="file://$(env MODELS_DIR)/rover/stl/wdisc.stl"/>
         </geometry>
+        <material name="gray">
+            <color rgba="0.4 0.4 0.4 1.0"/>
+        </material>
     </visual>
     <collision name='wheel_${index}_collision'>
         <geometry>
-            <cylinder radius="${diameter}" length="0.1"/>
+            <cylinder radius="${radius}" length="0.1"/>
         </geometry>
     </collision>
 </link>
+<link name="wheel_${index}_tyre">
+    <visual name="wheel_${index}_tyre_visual">
+        <geometry>
+            <mesh filename="file://$(env MODELS_DIR)/rover/stl/tyre.stl"/>
+        </geometry>
+        <material name="black">
+            <color rgba="0 0 0 1.0"/>
+        </material>
+    </visual>
+</link>
+<joint name="wheel_${index}_tyre_to_disc_joint" type="fixed">
+    <parent link="wheel_${index}_disc"/>
+    <child link="wheel_${index}_tyre"/>
+</joint>
 <joint name="wheel_${index}_joint" type="revolute">
     <parent link="base"/>
-    <child link="wheel_${index}"/>
-    <origin xyz="${xyz}" rpy="${pi/2} 0 0"/>
+    <child link="wheel_${index}_disc"/>
+    <origin xyz="${xyz}" rpy="${pi/2} 0 ${yaw}"/>
     <axis xyz="${axis}"/>
     <limit

Commit message: fix camera pose

File: src/simulation/models/rover/rover.xacro (robot description, xacro)
@@ -20,9 +20,4 @@
             <color rgba="0.4 0.4 0.4 1.0"/>
         </material>
-        <!--
-        <material name="blue">
-            <color rgba="0 0 0.7 1.0"/>
-        </material>
-        -->
     </visual>
     <collision name="base_collision">
@@ -122,5 +117,5 @@
     <parent link="base"/>
     <child link="camera"/>
-    <origin xyz="0 0 ${robot_side_z/2}"/>
+    <origin xyz="0 0 ${robot_side_z/2 + z_offset_to_center + 0.05}" rpy="0 0 0"/>
 </joint>
 <gazebo reference="camera">

File: src/simulation/models/rover/wheel.xacro (robot description, xacro)
@@ -10,6 +10,6 @@
             <mesh filename="file://$(env MODELS_DIR)/rover/stl/wdisc.stl"/>
         </geometry>
-        <material name="gray">
-            <color rgba="0.4 0.4 0.4 1.0"/>
+        <material name="white-ish">
+            <color rgba="0.7 0.7 0.7 1.0"/>
         </material>
     </visual>
