Commit message: add field world

File: src/simulation/models/objects/01-module/model.sdf.xacro (robot description, xacro)
@@ -3,38 +3,6 @@
 <model name="module">
 <pose>0 0 0 0 0 0</pose>
-<static>false</static>
-<xacro:include filename="$(env MODELS_DIR)/common/utils.xacro" />
-<link name="module_base">
-    <self_collide>false</self_collide>
-    <xacro:macro name="module_stl">
-        <geometry>
-            <mesh>
-                <uri>file:/$(env MODELS_DIR)/objects/01-module/01-module.stl</uri>
-                <scale>1 1 1</scale>
-            </mesh>
-        </geometry>
-    </xacro:macro>
-    <collision name="module_collision">
-        <xacro:module_stl/>
-    </collision>
-    <visual name="module_visual">
-        <xacro:module_stl/>
-        <material>
-            <script>
-                <uri>file://media/materials/scripts/gazebo.material</uri>
-                <name>Gazebo/Yellow</name>
-            </script>
-        </material>
-    </visual>
-    <xacro:cuboid_inertia pose="0.25 0.25 0.5 0 0 0" weight="100" a="0.5" b="0.5" c="1"/>
-</link>
-<include>
-    <uri>file:/$(env MODELS_DIR)/objects/main-panel</uri>
-    <pose>0.503 0 0.55 ${-pi/2} ${pi} ${-pi/2}</pose>
-</include>
-<joint name="main_panel_to_module_base_joint" type="fixed">
-    <parent>module_base</parent>
-    <child>main-panel::panel</child>
-</joint>
+<xacro:include filename="module.xacro" />
+<xacro:module suffix=""/>
 </model>
 </sdf>

File: src/simulation/models/objects/field/model.sdf.xacro (robot description, xacro)
@@ -1,29 +1,52 @@
 <?xml version="1.0" ?>
 <sdf xmlns:xacro="http://www.ros.org/wiki/xacro" version="1.10">
-  <model name="rc_terrain">
-    <pose>0 0 0 0 0 0</pose>
-    <static>true</static>
-    <link name="rc_terrain">
-      <xacro:macro name="terrain_stl">
-        <geometry>
-          <mesh>
-            <uri>file:/$(env MODELS_DIR)/objects/field/field-demo1.stl</uri>
-            <scale>1 1 1</scale>
-          </mesh>
-        </geometry>
-      </xacro:macro>
-      <collision name="terrain_collision">
-        <xacro:terrain_stl/>
-      </collision>
-      <visual name="terrain_visual">
-        <xacro:terrain_stl/>
-        <material>
-          <script>
-              <uri>file://media/materials/scripts/gazebo.material</uri>
-              <name>Gazebo/Grey</name>
-          </script>
-        </material>
-      </visual>
-    </link>
-  </model>
+<model name="rc_terrain">
+<pose>0 0 0 0 0 0</pose>
+<static>true</static>
+<link name="rc_terrain">
+  <xacro:macro name="terrain_stl">
+    <geometry>
+      <mesh>
+        <uri>file:/$(env MODELS_DIR)/objects/field/field-2024.stl</uri>
+        <scale>1 1 1</scale>
+      </mesh>
+    </geometry>
+  </xacro:macro>
+  <collision name="terrain_collision">
+    <xacro:terrain_stl/>
+  </collision>
+  <visual name="terrain_visual">
+    <xacro:terrain_stl/>
+    <material>
+      <script>
+          <uri>file://media/materials/scripts/gazebo.material</uri>
+          <name>Gazebo/Grey</name>
+      </script>
+    </material>
+  </visual>
+</link>
+<link name="fence">
+  <pose>10 10 0.15 0 0 0</pose>
+  <xacro:macro name="fence_stl">
+    <geometry>
+      <mesh>
+        <uri>file:/$(env MODELS_DIR)/objects/field/zabor.stl</uri>
+        <scale>1 1 1</scale>
+      </mesh>
+    </geometry>
+  </xacro:macro>
+  <collision name="fence_collision">
+    <xacro:fence_stl/>
+  </collision>
+  <visual name="fence_visual">
+    <xacro:fence_stl/>
+    <material>
+      <script>
+          <uri>file://media/materials/scripts/gazebo.material</uri>
+          <name>Gazebo/Black</name>
+      </script>
+    </material>
+  </visual>
+</link>
+</model>
 </sdf>

File: src/simulation/models/objects/main-panel/model.sdf.xacro (robot description, xacro)
@@ -3,137 +3,6 @@
 <model name="main-panel">
 <pose>0 0 0 0 0 0</pose>
-<static>false</static>
-<xacro:include filename="$(env MODELS_DIR)/common/utils.xacro" />
-<link name="panel">
-    <self_collide>false</self_collide>
-    <xacro:macro name="panel_stl">
-        <geometry>
-            <mesh>
-                <uri>file:/$(env MODELS_DIR)/objects/main-panel/main-panel.stl</uri>
-                <scale>1 1 1</scale>
-            </mesh>
-        </geometry>
-    </xacro:macro>
-    <collision name="panel_collision">
-        <xacro:panel_stl/>
-    </collision>
-    <visual name="panel_visual">
-        <xacro:panel_stl/>
-        <material>
-            <script>
-                <uri>file://media/materials/scripts/gazebo.material</uri>
-                <name>Gazebo/Yellow</name>
-            </script>
-        </material>
-    </visual>
-</link>
-<link name="panel_image">
-    <visual name="panel_image_visual">
-        <pose>0.35 0.225 0.005 0 0 0</pose>
-        <geometry>
-            <plane>
-                <size>0.7 0.45</size>
-            </plane>
-        </geometry>
-        <material>
-            <ambient>0.8 0.8 0.8 1</ambient>
-            <diffuse>0.8 0.8 0.8 1</diffuse>
-            <specular>1 0.8 0.8 1</specular>
-            <pbr>
-                <metal>
-                    <albedo_map>supply-texture.png</albedo_map>
-                    <normal_map>supply-texture.png</normal_map>
-                </metal>
-            </pbr>
-        </material>
-    </visual>
-</link>
-<joint name="pole_image_joint" type="fixed">
-    <parent>panel</parent>
-    <child>panel_image</child>
-</joint>
-<link name="panel_door">
-    <pose>0.46 0.16 -0.008 0 0 0</pose>
-    <self_collide>false</self_collide>
-    <xacro:macro name="panel_door_stl">
-        <geometry>
-            <mesh>
-                <uri>file:/$(env MODELS_DIR)/objects/main-panel/sampler-door.stl</uri>
-                <scale>1 1 1</scale>
-            </mesh>
-        </geometry>
-    </xacro:macro>
-    <collision name="panel_door_collision">
-        <xacro:panel_door_stl/>
-    </collision>
-    <visual name="panel_door_visual">
-        <xacro:panel_door_stl/>
-        <material>
-            <script>
-                <uri>file://media/materials/scripts/gazebo.material</uri>
-                <name>Gazebo/Blue</name>
-            </script>
-        </material>
-    </visual>
-</link>
-<joint name="panel_door_joint" type="prismatic">
-    <parent>panel</parent>
-    <child>panel_door</child>
-    <axis>
-        <xyz>-1 0 0</xyz>
-        <limit>
-            <lower>0</lower>
-            <upper>0.18</upper>
-        </limit>
-        <dynamics>
-            <damping>0</damping>
-            <spring_stiffness>0</spring_stiffness>
-            <spring_reference>0</spring_reference>
-        </dynamics>
-    </axis>
-    <physics>
-        <ode>
-            <cfm_damping>1</cfm_damping>
-        </ode>
-    </physics>
-</joint>
-<xacro:include filename="$(env MODELS_DIR)/objects/switch_rotate/rotator.xacro" />
-<xacro:include filename="$(env MODELS_DIR)/objects/switch/switch.xacro" />
-<xacro:include filename="$(env MODELS_DIR)/objects/button/button.xacro" />
-<xacro:include filename="$(env MODELS_DIR)/objects/weight-button/weight_button.xacro" />
-<xacro:include filename="$(env MODELS_DIR)/objects/switch_room/switch_room.xacro" />
-<xacro:macro name="trigger" params="type name pose">
-    <model name="${name}_trigger">
-        <pose>${pose}</pose>
-        <xacro:if value="${type == 'switch'}">
-            <xacro:switch name_prefix="${name}_"/>
-        </xacro:if>
-        <xacro:if value="${type == 'rotator'}">
-            <xacro:rotator name_prefix="${name}_"/>
-        </xacro:if>
-        <xacro:if value="${type == 'button'}">
-            <xacro:button name_prefix="${name}_"/>
-        </xacro:if>
-        <xacro:if value="${type == 'weight_button'}">
-            <xacro:weight_button name_prefix="${name}_"/>
-        </xacro:if>
-        <xacro:if value="${type == 'switch_room'}">
-            <xacro:switch_room name_prefix="${name}_"/>
-        </xacro:if>
-    </model>
-    <joint name="${name}_trigger_to_wall_joint" type="fixed">
-        <parent>panel</parent>
-        <child>${name}_trigger::${name}_frame</child>
-    </joint>
-</xacro:macro>
-<xacro:trigger type="rotator" name="door_rotator" pose="0.53 0.095 0 0 0 0"/>
-<xacro:trigger type="weight_button" name="secret-button" pose="0.55 0.16 -0.06 ${-pi/2} 0 0"/>
-<xacro:trigger type="switch_room" name="switch_room" pose="0.16 0.29 0 0 0 ${-pi/2}"/>
-<xacro:trigger type="button" name="button-1" pose="0.291 0.289 0 0 0 0"/>
-<xacro:trigger type="switch" name="switch-1" pose="0.133 0.115 0 0 0 ${-pi/2}"/>
-<xacro:trigger type="switch" name="switch-2" pose="0.193 0.115 0 0 0 ${-pi/2}"/>
-<xacro:trigger type="switch" name="switch-3" pose="0.253 0.115 0 0 0 ${-pi/2}"/>
-<xacro:trigger type="switch" name="switch-4" pose="0.313 0.115 0 0 0 ${-pi/2}"/>
-<xacro:trigger type="switch" name="switch-5" pose="0.373 0.115 0 0 0 ${-pi/2}"/>
+<xacro:include filename="main-panel.xacro" />
+<xacro:main_panel suffix=""/>
 </model>
 </sdf>

File: src/simulation/models/objects/marker/model.sdf.xacro (robot description, xacro)
@@ -3,54 +3,6 @@
 <model name="marker_pole">
 <pose>0 0 0 0 0 0</pose>
-<static>true</static>
-<link name="marker_pole">
-  <collision name="pole_collision">
-    <geometry>
-      <box>
-        <size>0.3 0.3 0.7</size>
-      </box>
-    </geometry>
-  </collision>
-  <visual name="pole_visual">
-    <pose>0 0 0.35 ${pi} 0 0</pose>
-    <geometry>
-      <mesh>
-        <uri>file:/$(env MODELS_DIR)/objects/marker/marker10.stl</uri>
-        <scale>1 1 1</scale>
-      </mesh>
-    </geometry>
-    <material>
-      <script>
-        <uri>file://media/materials/scripts/gazebo.material</uri>
-        <name>Gazebo/Yellow</name>
-      </script>
-    </material>
-  </visual>
-</link>
-<link name="marker_image">
-  <visual name="marker_image_visual">
-    <pose>-0.15 0 0.175 ${pi/2} 0 ${-pi/2}</pose>
-    <geometry>
-      <plane>
-        <size>0.2 0.3</size>
-      </plane>
-    </geometry>
-    <material>
-      <ambient>0.8 0.8 0.8 1</ambient>
-      <diffuse>0.8 0.8 0.8 1</diffuse>
-      <specular>1 0.8 0.8 1</specular>
-      <pbr>
-          <metal>
-            <albedo_map>10.png</albedo_map>
-            <normal_map>10.png</normal_map>
-          </metal>
-        </pbr>
-    </material>
-  </visual>
-</link>
-<joint name="pole_image_joint" type="fixed">
-  <parent>marker_pole</parent>
-  <child>marker_image</child>
-</joint>
+<xacro:include filename="marker.xacro" />
+<xacro:marker/>
 </model>
 </sdf>

File: src/simulation/models/worlds/field/field.sdf.xacro (robot description, xacro)
@@ -1,31 +1,86 @@
 <?xml version="1.0" ?>
 <sdf xmlns:xacro="http://www.ros.org/wiki/xacro" version="1.10">
-<world name="field_world">
+<world name="plane_world">
 <xacro:include filename="$(env MODELS_DIR)/common/plugins.xacro" />
 <xacro:include filename="$(env MODELS_DIR)/common/simple_light.xacro" />
+<xacro:include filename="$(env MODELS_DIR)/common/utils.xacro" />
+<xacro:include filename="$(env MODELS_DIR)/objects/marker/marker.xacro" />
+<xacro:include filename="$(env MODELS_DIR)/objects/01-module/module.xacro" />
 <include>
     <uri>file:/$(env MODELS_DIR)/objects/field</uri>
-    <pose>0 0 0 ${-pi/2} 0 0</pose>
+    <pose>0 0 0 0 0 0</pose>
 </include>
-<include>
-    <name>pole_1</name>
-    <uri>file:/$(env MODELS_DIR)/objects/marker</uri>
-    <pose>5 0 1 0 0 0</pose>
-</include>
-<include>
-    <name>pole_2</name>
-    <uri>file:/$(env MODELS_DIR)/objects/marker</uri>
-    <pose>0 5 1 0 0 0</pose>
-</include>
+<model name='explorer'>
+    <include>
+         <uri>file:/$(env MODELS_DIR)/explorer/explorer.urdf</uri>
+         <pose>5.0 5.0 0.5 0.0 0 0.0</pose>
+    </include>
+</model>
 <include>
     <uri>file:/$(env MODELS_DIR)/objects/garage</uri>
-    <pose>0 -8 0 0 0 ${pi}</pose>
+    <pose>18.068 5.732 0.1 0 0 -2.55</pose>
 </include>
-<model name='rover'>
-    <include>
-         <uri>file:/$(env MODELS_DIR)/rover/rover.urdf</uri>
-         <pose>0.0 0.0 0.5 0.0 0 0.0</pose>
-    </include>
-</model>
+<joint name="garage_to_world" type="fixed">
+    <parent>world</parent>
+    <child>garage::garage</child>
+</joint>
+<xacro:macro name="garage_door_trigger" params="name force">
+    <plugin
+        filename="${gazebo_systems_lib_dir}/libTriggerSystems.so"
+        name="trigger_systems::DoorButton">
+        <hinge_joint>garage_door_joint</hinge_joint>
+        <trigger_joint>${name}_button_to_frame_joint</trigger_joint>
+        <percentage_activated>50</percentage_activated>
+        <opening_force>${force}</opening_force>
+        <closing_force>0</closing_force>
+        <is_oneshot>true</is_oneshot>
+        <log_name>${name}</log_name>
+        <do_log>false</do_log>
+    </plugin>
+</xacro:macro>
+<xacro:garage_door_trigger name="outer_open" force="5000"/>
+<xacro:garage_door_trigger name="outer_close" force="-5000"/>
+<xacro:garage_door_trigger name="inner_open" force="5000"/>
+<xacro:garage_door_trigger name="inner_close" force="-5000"/>
+<xacro:macro name="world_module" params="suffix pose">
+    <model name='module_${suffix}'>
+        <xacro:module suffix="${suffix}"/>
+        <pose>${pose}</pose>
+    </model>
+    <joint name="module_${suffix}_to_world" type="fixed">
+        <parent>world</parent>
+        <child>module_${suffix}::module_base</child>
+    </joint>
+    <plugin
+        filename="${gazebo_systems_lib_dir}/libTriggerSystems.so"
+        name="trigger_systems::DoorButton">
+        <hinge_joint>${suffix}_panel_door_joint</hinge_joint>
+        <trigger_joint>${suffix}_door_rotator_rotator_to_frame_joint</trigger_joint>
+        <percentage_activated>50</percentage_activated>
+        <opening_force>100</opening_force>
+        <closing_force>-100</closing_force>
+        <is_oneshot>true</is_oneshot>
+        <log_name>${suffix}_panel_door</log_name>
+        <do_log>true</do_log>
+    </plugin>
+</xacro:macro>
+<!--
+<xacro:world_module suffix="outter" pose="3.346 12.598 1.0 0 0 1.57"/>
+<xacro:world_module suffix="inner" pose="16.066 1.065 0.5 0 0 0.93"/>
+-->
+<xacro:macro name="pole" params="index pose image">
+    <model name='pole_${index}'>
+        <xacro:marker image="${image}"/>
+        <pose>${pose}</pose>
+    </model>
+</xacro:macro>
+<xacro:property name="pole_z_offset" value="-0.175"/>
+<xacro:pole index="0" pose="14.2 4 ${pole_z_offset + 0.7} 0 0 0" image="31.png"/>
+<xacro:pole index="1" pose="15.7 14.6 ${pole_z_offset + 2.2} 0 0 0" image="32.png"/>
+<xacro:pole index="2" pose="9 10 ${pole_z_offset + 1.15} 0 0 0" image="33.png"/>
+<xacro:pole index="3" pose="7 16.5 ${pole_z_offset + 1.9} 0 0 0" image="34.png"/>
+<xacro:pole index="4" pose="2.5 3.7 ${pole_z_offset + 1.65} 0 0 0" image="35.png"/>
+<xacro:pole index="5" pose="1.3 9.7 ${pole_z_offset + 0.9} 0 0 0" image="36.png"/>
+<xacro:pole index="6" pose="1 19 ${pole_z_offset + 1.6} 0 0 0" image="37.png"/>
 </world>
 </sdf>
