Commit message: improve rover

File: src/simulation/models/explorer/explorer.urdf.xacro (robot description, xacro)
@@ -6,5 +6,5 @@
     <parent link="base"/>
     <child link="base_link"/>
-    <origin rpy="0 0 0" xyz="0 0 0.215"/>
+    <origin rpy="0 0 0" xyz="0.2 0 0.251"/>
 </joint>
 <gazebo>

File: src/simulation/models/rover/rover.xacro (robot description, xacro)
@@ -112,4 +112,34 @@
 <xacro:wheel index="2" xyz="${wheel_x_offset} ${wheel_y_offset} 0" yaw="${pi}" axis="0 0 1" radius="${wheel_radius}"/>
 <xacro:wheel index="3" xyz="${-wheel_x_offset} ${wheel_y_offset} 0" yaw="${pi}" axis="0 0 1" radius="${wheel_radius}"/>
+<link name="mount_plate">
+    <visual name="mount_plate_visual">
+        <geometry>
+            <mesh filename="file://$(env MODELS_DIR)/rover/stl/moun-plate.stl"/>
+        </geometry>
+        <material name="wood">
+            <color rgba="0.7 0.7 0.7 1.0"/>
+        </material>
+    </visual>
+</link>
+<joint name="mount_plate_to_base" type="fixed">
+    <parent link="base"/>
+    <child link="mount_plate"/>
+    <origin xyz="0 0 0" rpy="0 0 0"/>
+</joint>
+<link name="realsense">
+    <visual name="realsense_visual">
+        <geometry>
+            <mesh filename="file://$(env MODELS_DIR)/rover/stl/realsens.stl"/>
+        </geometry>
+        <material name="steel">
+            <color rgba="0.8 0.8 0.8 1.0"/>
+        </material>
+    </visual>
+</link>
+<joint name="realsense_to_base" type="fixed">
+    <parent link="base"/>
+    <child link="realsense"/>
+    <origin xyz="0 0 0" rpy="0 0 0"/>
+</joint>
 <!-- CAMERA BLOCK-->
 <link name="camera"></link>
@@ -117,5 +147,5 @@
     <parent link="base"/>
     <child link="camera"/>
-    <origin xyz="0 0 ${robot_side_z/2 + z_offset_to_center + 0.05}" rpy="0 0 0"/>
+    <origin xyz="0.363 0 0.216" rpy="0 -0.17 0"/>
 </joint>
 <gazebo reference="camera">

File: src/simulation/models/worlds/field/field.sdf.xacro (robot description, xacro)
@@ -14,5 +14,5 @@
     <include>
          <uri>file:/$(env MODELS_DIR)/explorer/explorer.urdf</uri>
-         <pose>5.0 5.0 0.5 0.0 0 0.0</pose>
+         <pose>10 11 0.5 0.0 0 0.0</pose>
     </include>
 </model>

Commit message: add cameras to rover and sample_can

File: src/simulation/models/explorer/explorer.urdf.xacro (robot description, xacro)
@@ -3,4 +3,5 @@
 <xacro:include filename="$(env MODELS_DIR)/rover/rover.urdf.xacro" />
 <xacro:include filename="$(find ruka_gz)/config/ruka_gz.urdf.xacro" />
+<xacro:include filename="$(env MODELS_DIR)/objects/cameras/d435.xacro" />
 <joint name="ruka_to_rover" type="fixed">
     <parent link="base"/>

File: src/simulation/models/rover/rover.xacro (robot description, xacro)
@@ -127,45 +127,49 @@
     <origin xyz="0 0 0" rpy="0 0 0"/>
 </joint>
-<link name="realsense">
-    <visual name="realsense_visual">
-        <geometry>
-            <mesh filename="file://$(env MODELS_DIR)/rover/stl/realsens.stl"/>
-        </geometry>
-        <material name="steel">
-            <color rgba="0.8 0.8 0.8 1.0"/>
-        </material>
-    </visual>
-</link>
-<joint name="realsense_to_base" type="fixed">
-    <parent link="base"/>
-    <child link="realsense"/>
+<!-- CAMERA BLOCK-->
+<xacro:include filename="$(env MODELS_DIR)/objects/cameras/d435.xacro" />
+<xacro:include filename="$(env MODELS_DIR)/objects/cameras/fov120.xacro" />
+<link name="realsense_mount">
+    <visual name="realsense_mount_visual">
+        <geometry>
+            <mesh filename="file://$(env MODELS_DIR)/rover/stl/d435-mount.stl"/>
+        </geometry>
+        <material name="mount-color">
+            <color rgba="0.2 0.2 0.2 1.0"/>
+        </material>
+    </visual>
+</link>
+<joint name="realsense_mount_to_base" type="fixed">
+    <parent link="base"/>
+    <child link="realsense_mount"/>
     <origin xyz="0 0 0" rpy="0 0 0"/>
 </joint>
-<!-- CAMERA BLOCK-->
-<link name="camera"></link>
-<joint name="camera_joint" type="fixed">
-    <parent link="base"/>
-    <child link="camera"/>
-    <origin xyz="0.363 0 0.216" rpy="0 -0.17 0"/>
-</joint>
-<gazebo reference="camera">
-    <sensor name="camera" type="camera">
-        <camera>
-            <horizontal_fov>1.047</horizontal_fov>
-            <image>
-                <width>320</width>
-                <height>240</height>
-            </image>
-            <clip>
-                <near>0.1</near>
-                <far>100</far>
-            </clip>
-        </camera>
-        <always_on>1</always_on>
-        <update_rate>30</update_rate>
-        <visualize>true</visualize>
-        <topic>camera</topic>
-    </sensor>
-</gazebo>
+<xacro:realsense-d435 suffix="_front"/>
+<joint name="realsense_d435_front_frame_to_base" type="fixed">
+    <parent link="base"/>
+    <child link="realsense_d435_front_frame"/>
+    <origin xyz="0.339 0 0.223344" rpy="${-pi/2} 0 -0.09"/>
+</joint>
+<link name="top_mount">
+    <visual name="top_mount_visual">
+        <geometry>
+            <mesh filename="file://$(env MODELS_DIR)/rover/stl/cam120-stoika.stl"/>
+        </geometry>
+        <material name="mount-color">
+            <color rgba="0.2 0.2 0.2 1.0"/>
+        </material>
+    </visual>
+</link>
+<joint name="top_mount_to_base" type="fixed">
+    <parent link="base"/>
+    <child link="top_mount"/>
+    <origin xyz="0 0 0" rpy="0 0 0"/>
+</joint>
+<xacro:camera-fov120 suffix="_top"/>
+<joint name="fov120_top_frame_to_base" type="fixed">
+    <parent link="base"/>
+    <child link="fov120_top_frame"/>
+    <origin xyz="-0.315 0 0.8788" rpy="0 0.175 0"/>
+</joint>
 <!-- END CAMERA BLOCK-->
 <gazebo>

File: src/simulation/models/worlds/field/field.sdf.xacro (robot description, xacro)
@@ -83,4 +83,8 @@
 <xacro:pole index="5" pose="1.3 9.7 ${pole_z_offset + 0.9} 0 0 0" image="36.png"/>
 <xacro:pole index="6" pose="1 19 ${pole_z_offset + 1.6} 0 0 0" image="37.png"/>
+<include>
+    <uri>file:/$(env MODELS_DIR)/objects/sample_can</uri>
+    <pose>15.88784329 1.74618694 0.992 0 0 0</pose>
+</include>
 </world>
 </sdf>
