Commit message: cylinder colider for sample can

File: src/simulation/models/objects/sample_can/model.sdf.xacro (robot description, xacro)
@@ -15,5 +15,10 @@
     </xacro:macro>
     <collision name="can_collision">
-        <xacro:can_stl/>
+        <geometry>
+            <cylinder>
+                <radius>0.05</radius>
+                <length>0.1</length>
+            </cylinder>
+        </geometry>
     </collision>
     <visual name="can_visual">

File: src/simulation/models/worlds/field/field.sdf.xacro (robot description, xacro)
@@ -65,8 +65,6 @@
     </plugin>
 </xacro:macro>
-<!--
 <xacro:world_module suffix="outter" pose="3.346 12.598 1.0 0 0 1.57"/>
 <xacro:world_module suffix="inner" pose="16.066 1.065 0.5 0 0 0.93"/>
--->
 <xacro:macro name="pole" params="index pose image">
     <model name='pole_${index}'>
